File: matronome.kicad_sch (KiCad schematic)
At the start: 8 parts

Commit message: add rotary encoder
Parts:
- added SW?: RotaryEncoder, symbol Device:RotaryEncoder
Connections:
- net at U?.11 (PD6): now also SW?.B
- net at U?.8 (PD4): now also SW?.A
- net at U?.9 (PD5): now also SW?.C
Changed lines of the file:
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@@
     (pin "2")
+  )
+  (symbol (lib_id "Device:RotaryEncoder") (at 161.29 125.73 0) (unit 1)
+    (in_bom yes) (on_board yes) (fields_autoplaced)
+    (property "Reference" "SW?" (id 0) (at 167.64 124.4599 0)
+      (effects (font (size 1.27 1.27)) (justify left))
+    )
+    (property "Value" "RotaryEncoder" (id 1) (at 167.64 126.9999 0)
+      (effects (font (size 1.27 1.27)) (justify left))
+    )
+    (property "Footprint" "" (id 2) (at 157.48 121.666 0)
+      (effects (font (size 1.27 1.27)) hide)
+    )
+    (property "Datasheet" "~" (id 3) (at 161.29 119.126 0)
+      (effects (font (size 1.27 1.27)) hide)
+    )
+    (pin "A")
+    (pin "B")
+    (pin "C")
   )
   (sheet_instances
@@
       (reference "SW?") (unit 1) (value "SW_SPST") (footprint "")
     )
+    (path "/f879c0e8-5893-4eb4-8e59-2292a632100f"
+      (reference "SW?") (unit 1) (value "RotaryEncoder") (footprint "")
+    )
     (path "/67763d19-f622-4e1e-81e5-5b24da7c3f99"
